File: klon.kicad_pcb (KiCad board)
At the start: 2 copper layers, 60 x 100 mm, 71 parts, among them SW1 SW_DPDT_x2, U1 TL072, U2 LTC1044, U3 TL072

Commit message: update pcb layout
Parts:
- removed GAIN_1: 100K, Connector_PinHeader_2.54mm:PinHeader_2x03_P2.54mm_Vertical
- added GAIN: 100K, Connector_PinHeader_2.54mm:PinHeader_2x03_P2.54mm_Vertical, B.Cu at (51.5, 120.5)
- moved D6 0.50 mm to (97.7, 132.0)
- renumbered D3_ON1 to D3_ON, D4_OFF1 to D4_OFF, D5_CLIP1 to D5, D6_CLIP1 to D6, SW1 to SW, TONE1 to TONE, VOL1 to VOL
Routing:
- net +9V: track 0.00 -> 329.1 mm, vias 0 -> 2
- net /+4.5V: track 0.00 -> 226.7 mm, vias 0 -> 2
- net Net-(OUT1-PadT): track 0.00 -> 131.4 mm
- net Net-(C18-Pad1): track 0.00 -> 97.6 mm
- net /-8.6V: track 0.00 -> 96.1 mm, vias 0 -> 5
- net Net-(R26-Pad1): track 0.00 -> 92.0 mm, vias 0 -> 2
- net Net-(R30-Pad2): track 0.00 -> 87.2 mm, vias 0 -> 1
- net Net-(C8-Pad1): track 0.00 -> 84.7 mm
- net Net-(C1-Pad1): track 0.00 -> 72.6 mm
- net Net-(C5-Pad2): track 0.00 -> 71.7 mm, vias 0 -> 2
- net Net-(C19-Pad1): track 0.00 -> 69.9 mm
- net Net-(D4_OFF1-Pad2): track 0.00 -> 59.6 mm
- net Net-(C16-Pad2): track 0.00 -> 58.3 mm, vias 0 -> 2
- net Net-(GAIN_1-Pad6): track 0.00 -> 57.7 mm
- net /+16.2V: track 0.00 -> 56.8 mm, vias 0 -> 2
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- added copper zone on B.Cu, net GND
- added copper zone on F.Cu, net GND
Other:
- board text added: "Cosmik Debris"
- board text added: "v0.1.0"
